Commit message: update

File: src/robot_description/urdf/robot.urdf (robot description, URDF)
Before this commit: robot robot, 16 links, 15 joints
Links:
- added link roda_direita, mass 0.01; collision sphere radius=0.02; visual sphere radius=0.02
- added link roda_esquerda, mass 0.01; collision sphere radius=0.02; visual sphere radius=0.02
- added link roda_frente, mass 0.01; collision sphere radius=0.02; visual sphere radius=0.02
- added link roda_tras, mass 0.01; collision sphere radius=0.02; visual sphere radius=0.02
- link antebraco_direito: mass 0.2 -> 0.05
- link antebraco_esquerdo: mass 0.2 -> 0.05
- link base_link: mass 10.0 -> 15.0
- link coluna: mass 0.5 -> 0.2
- link cotovelo_direito: mass 0.1 -> 0.05
- link cotovelo_esquerdo: mass 0.1 -> 0.05
- link ombro_direito: mass 0.1 -> 0.05
- link ombro_esquerdo: mass 0.1 -> 0.05
- link torso: mass 0.8 -> 0.2
Joints:
- added joint roda_direita_base_link: type fixed, parent base_link, child roda_direita, origin xyz=0.0 -0.10 -0.02 rpy=0 0 0, axis 0 1 0
- added joint roda_esquerda_base_link: type fixed, parent base_link, child roda_esquerda, origin xyz=0.0 0.10 -0.02 rpy=0 0 0, axis 0 1 0
- added joint roda_frente_base_link: type fixed, parent base_link, child roda_frente, origin xyz=0.10 0.0 -0.02 rpy=0 0 0, axis 0 1 0
- added joint roda_tras_base_link: type fixed, parent base_link, child roda_tras, origin xyz=-0.10 0.0 -0.02 rpy=0 0 0, axis 0 1 0
